File: selen-full/selen-full.kicad_sch (KiCad schematic)
At the start: 36 parts, among them J1 AudioJack4, SW1 SW_Push, SW10 SW_Push, SW11 SW_Push, SW12 SW_Push, SW13 SW_Push, SW14 SW_Push, SW15 SW_Push, SW16 SW_Push, SW17 SW_Push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

Commit message: Update
Parts:
- D1, D10, D11, D12, D13, D14, D15, D16, D17, D2, D3, D4, D5, D6, D7, D8, D9: value D -> (none); footprint selen:D_SOD-123_axial -> (none)
- J1: value AudioJack4 -> (none); footprint kbd:MJ-4PP-9 -> (none)
- SW1, SW10, SW11, SW12, SW13, SW14, SW15, SW16, SW17, SW2, SW3, SW4, SW5, SW6, SW7, SW8, SW9: value SW_Push -> (none); footprint kbd:CherryMX_Choc_Hotswap -> (none)
- U1: value XIAO-RP2040 -> (none); footprint selen:XIAO-MOUDLE14P-2.54-21X17.8MM_SMD_reversible -> (none)
Connections:
- net +3V3: now also J1.C
- net GND: no longer J1.C
